File: Hardware/DigitalSynthCape/DigitalSynthCape.kicad_sch (KiCad schematic)
At the start: 11 parts, among them P9 BeagleBone_Black_Header, SW1 SW_DIP_x02, U1 CAT24C256

Commit message: Added Render
Parts:
- RV1: footprint (none) -> Potentiometer_THT:Potentiometer_Bourns_PTA1543_Single_Slide
Changed lines of the file:
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@@
       (effects (font (size 1.27 1.27)) (justify right))
     )
-    (property "Footprint" "" (at 109.22 54.61 0)
+    (property "Footprint" "Potentiometer_THT:Potentiometer_Bourns_PTA1543_Single_Slide" (at 109.22 54.61 0)
       (effects (font (size 1.27 1.27)) hide)
     )
