File: Hardware/DigitalSynthCape/DigitalSynthCape.kicad_sch (KiCad schematic)
At the start: 20 parts, among them J1 Conn_01x01_Male, P9 BeagleBone_Black_Header

Commit message: Updates
Parts:
- removed RV1: R_Potentiometer, Potentiometer_THT:Potentiometer_Bourns_PTA1543_Single_Slide, symbol Device:R_Potentiometer
- added R18: COM-09806, Project:TRIM_COM-09806, symbol COM-09806:COM-09806
- J1: footprint Connector_Samtec_HPM_THT:Samtec_HPM-01-01-x-S_Straight_1x01_Pitch5.08mm -> Connector_Pin:Pin_D1.0mm_L10.0mm
Connections:
- net +1V8: now also R18.1
- net AIN0: now also R2.2
- net AIN1: now also R18.2
- net GNDA: now also R18.3
- net Key2: now also R2.1
Changed lines of the file:
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@@
+    (stroke (width 0) (type solid))
+  )
+  (wire (pts (xy 166.37 96.52) (xy 166.37 104.14))
     (stroke (width 0) (type solid))
   )
@@
     (stroke (width 0) (type solid))
   )
+  (wire (pts (xy 173.99 91.44) (xy 179.07 91.44))
+    (stroke (width 0) (type solid))
+  )
   (wire (pts (xy 179.07 119.38) (xy 179.07 129.54))
     (stroke (width 0) (type default))
@@
     (stroke (width 0) (type solid))
   )
+  (wire (pts (xy 179.07 91.44) (xy 179.07 96.52))
+    (stroke (width 0) (type solid))
+  )
   (wire (pts (xy 38.1 80.01) (xy 57.15 80.01))
     (stroke (width 0) (type solid))
@@
     (stroke (width 0) (type default))
   )
+  (wire (pts (xy 153.67 88.9) (xy 153.67 91.44))
+    (stroke (width 0) (type default))
+  )
   (wire (pts (xy 38.1 59.69) (xy 57.15 59.69))
     (stroke (width 0) (type solid))
@@
   )
   (wire (pts (xy 135.89 119.38) (xy 135.89 129.54))
+    (stroke (width 0) (type default))
+  )
+  (wire (pts (xy 153.67 91.44) (xy 158.75 91.44))
     (stroke (width 0) (type default))
   )
@@
   (label "Key12" (at 223.52 119.38 270) (fields_autoplaced)
     (effects (font (size 1.27 1.27)) (justify right bottom))
+  )
+  (label "AIN1" (at 166.37 104.14 90) (fields_autoplaced)
+    (effects (font (size 1.27 1.27)) (justify left bottom))
   )
   (label "GPIO48" (at 38.1 46.99 0) (fields_autoplaced)
@@
     )
   )
+  (symbol (lib_id "Resistors:R") (at 135.89 133.35 0) (unit 1)
+    (in_bom yes) (on_board yes) (dnp no) (fields_autoplaced)
+    (property "Reference" "R2" (at 138.43 132.08 0)
+      (effects (font (size 1.27 1.27)) (justify left))
+    )
+    (property "Value" "R" (at 138.43 134.62 0)
+      (effects (font (size 1.27 1.27)) (justify left))
+    )
+    (property "Footprint" "Resistor_SMD:R_1206_3216Metric" (at 135.89 152.4 0)
+      (effects (font (size 1.27 1.27)) hide)
+    )
+    (property "Datasheet" "" (at 134.62 147.32 0)
+      (effects (font (size 1.27 1.27)) hide)
+    )
+    (pin "1")
+    (pin "2")
+    (instances
+      (project "DigitalSynthCape"
+        (path "/e63e39d7-6ac0-4ffd-8aa3-1841a4541b55"
+          (reference "R2") (unit 1)
+        )
+      )
+    )
+  )
   (symbol (lib_id "Resistors:R") (at 187.96 133.35 0) (unit 1)
     (in_bom yes) (on_board yes) (dnp no) (fields_autoplaced)
@@
       (effects (font (size 1.27 1.27)))
     )
-    (property "Footprint" "Connector_Samtec_HPM_THT:Samtec_HPM-01-01-x-S_Straight_1x01_Pitch5.08mm" (at 118.11 102.87 0)
+    (property "Footprint" "Connector_Pin:Pin_D1.0mm_L10.0mm" (at 118.11 102.87 0)
       (effects (font (size 1.27 1.27)) hide)
     )
@@
     )
   )
-  (symbol (lib_id "Resistors:R") (at 135.8681 133.3196 0) (unit 1)
-    (in_bom yes) (on_board yes) (dnp no) (fields_autoplaced)
-    (property "Reference" "R2" (at 138.4081 132.0496 0)
-      (effects (font (size 1.27 1.27)) (justify left))
-    )
-    (property "Value" "R" (at 138.4081 134.5896 0)
-      (effects (font (size 1.27 1.27)) (justify left))
-    )
-    (property "Footprint" "Resistor_SMD:R_1206_3216Metric" (at 135.8681 152.3696 0)
-      (effects (font (size 1.27 1.27)) hide)
-    )
-    (property "Datasheet" "" (at 134.5981 147.2896 0)
-      (effects (font (size 1.27 1.27)) hide)
-    )
-    (pin "1")
-    (pin "2")
-    (instances
-      (project "DigitalSynthCape"
-        (path "/e63e39d7-6ac0-4ffd-8aa3-1841a4541b55"
-          (reference "R2") (unit 1)
+  (symbol (lib_id "COM-09806:COM-09806") (at 166.37 91.44 0) (unit 1)
+    (in_bom yes) (on_board yes) (dnp no) (fields_autoplaced)
+    (property "Reference" "R18" (at 166.37 85.09 0)
+      (effects (font (size 1.27 1.27)))
+    )
+    (property "Value" "COM-09806" (at 166.37 87.63 0)
+      (effects (font (size 1.27 1.27)))
+    )
+    (property "Footprint" "Project:TRIM_COM-09806" (at 166.37 91.44 0)
+      (effects (font (size 1.27 1.27)) (justify bottom) hide)
+    )
+    (property "Datasheet" "" (at 166.37 91.44 0)
+      (effects (font (size 1.27 1.27)) hide)
+    )
+    (property "PARTREV" "N/A" (at 166.37 91.44 0)
+      (effects (font (size 1.27 1.27)) (justify bottom) hide)
+    )
+    (property "STANDARD" "Manufacturer Recommendations" (at 166.37 91.44 0)
+      (effects (font (size 1.27 1.27)) (justify bottom) hide)
+    )
+    (property "MAXIMUM_PACKAGE_HEIGHT" "5.08 mm" (at 166.37 91.44 0)
+      (effects (font (size 1.27 1.27)) (justify bottom) hide)
+    )
+    (property "MANUFACTURER" "Sparkfun" (at 166.37 91.44 0)
+      (effects (font (size 1.27 1.27)) (justify bottom) hide)
+    )
+    (pin "2")
+    (pin "3")
+    (pin "1")
+    (instances
+      (project "DigitalSynthCape"
+        (path "/e63e39d7-6ac0-4ffd-8aa3-1841a4541b55"
+          (reference "R18") (unit 1)
+        )
+      )
+    )
+  )
+  (symbol (lib_id "power:+1V8") (at 153.67 88.9 0) (mirror y) (unit 1)
+    (in_bom yes) (on_board yes) (dnp no)
+    (property "Reference" "#PWR01" (at 153.67 92.71 0)
+      (effects (font (size 1.27 1.27)) hide)
+    )
+    (property "Value" "+1V8" (at 153.3144 85.852 90)
+      (effects (font (size 1.27 1.27)) (justify left))
+    )
+    (property "Footprint" "" (at 153.67 88.9 0)
+      (effects (font (size 1.27 1.27)) hide)
+    )
+    (property "Datasheet" "" (at 153.67 88.9 0)
+      (effects (font (size 1.27 1.27)) hide)
+    )
+    (pin "1")
+    (instances
+      (project "DigitalSynthCape"
+        (path "/e63e39d7-6ac0-4ffd-8aa3-1841a4541b55"
+          (reference "#PWR01") (unit 1)
         )
       )
@@
     )
   )
+  (symbol (lib_id "power:GNDA") (at 179.07 96.52 0) (unit 1)
+    (in_bom yes) (on_board yes) (dnp no)
+    (property "Reference" "#PWR02" (at 179.07 102.87 0)
+      (effects (font (size 1.27 1.27)) hide)
+    )
+    (property "Value" "GNDA" (at 179.1843 100.8444 0)
+      (effects (font (size 1.27 1.27)))
+    )
+    (property "Footprint" "" (at 179.07 96.52 0)
+      (effects (font (size 1.27 1.27)) hide)
+    )
+    (property "Datasheet" "" (at 179.07 96.52 0)
+      (effects (font (size 1.27 1.27)) hide)
+    )
+    (pin "1")
+    (instances
+      (project "DigitalSynthCape"
+        (path "/e63e39d7-6ac0-4ffd-8aa3-1841a4541b55"
+          (reference "#PWR02") (unit 1)
+        )
+      )
+    )
+  )
   (symbol (lib_id "Resistors:R") (at 128.27 133.35 0) (unit 1)
     (in_bom yes) (on_board yes) (dnp no) (fields_autoplaced)
@@
         )
       )
-    )
-  )
-  (symbol (lib_id "Device:R_Potentiometer") (at 124.46 38.1 0) (unit 1)
-    (in_bom yes) (on_board yes) (dnp no) (fields_autoplaced)
-    (property "Reference" "RV1" (at 121.92 36.83 0)
-      (effects (font (size 1.27 1.27)) (justify right))
-    )
-    (property "Value" "R_Potentiometer" (at 121.92 39.37 0)
-      (effects (font (size 1.27 1.27)) (justify right))
-    )
-    (property "Footprint" "Potentiometer_THT:Potentiometer_Bourns_PTA1543_Single_Slide" (at 124.46 38.1 0)
-      (effects (font (size 1.27 1.27)) hide)
-    )
-    (property "Datasheet" "~" (at 124.46 38.1 0)
-      (effects (font (size 1.27 1.27)) hide)
-    )
-    (pin "3")
-    (pin "2")
-    (pin "1")
-    (instances
-      (project "DigitalSynthCape"
-        (path "/e63e39d7-6ac0-4ffd-8aa3-1841a4541b55"
-          (reference "RV1") (unit 1)
-        )
-      )

Commit message: Updates to Readme
Other:
- note added: "1.8 Volt Reference"
- note added: "A Beagle Bone Black Cape"
- note added: "Beagle Bone Connector"
- note added: "Keys"
- note added: "Secondary Potentiometer"
- note added: "This is what you connect to the various notes"
- note added: "[1] Keyboard Cape"
- moved on the sheet: J1, P9, R1, R10, R11, R12, R13, R14, R15, R16, R17, R18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
