File: Hardware/DigitalSynthCape/DigitalSynthCape.kicad_pcb (KiCad board)
At the start: 2 copper layers, 86.4 x 54.6 mm, 23 parts, among them J10 Key 9, J11 Key 10, J12 Key 11, J13 Key 12, J14 Key 13, J15 Key 14, J16 Key 15, J17 Key 16, J18 Key 17, J2 Key 1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

Commit message: Added Render
Parts:
- removed J10: Key 9, TestPoint:TestPoint_Pad_1.0x1.0mm
- removed J11: Key 10, TestPoint:TestPoint_Pad_1.0x1.0mm
- removed J12: Key 11, TestPoint:TestPoint_Pad_1.0x1.0mm
- removed J13: Key 12, TestPoint:TestPoint_Pad_1.0x1.0mm
- removed J14: Key 13, TestPoint:TestPoint_Pad_1.0x1.0mm
- removed J15: Key 14, TestPoint:TestPoint_Pad_1.0x1.0mm
- removed J16: Key 15, TestPoint:TestPoint_Pad_1.0x1.0mm
- removed J17: Key 16, TestPoint:TestPoint_Pad_1.0x1.0mm
- removed J18: Key 17, TestPoint:TestPoint_Pad_1.0x1.0mm
- removed J2: Key 1, TestPoint:TestPoint_Pad_1.0x1.0mm
- removed J3: Key 2, TestPoint:TestPoint_Pad_1.0x1.0mm
- removed J4: Key 3, TestPoint:TestPoint_Pad_1.0x1.0mm
- removed J5: Key 4, TestPoint:TestPoint_Pad_1.0x1.0mm
- removed J6: Key 5, TestPoint:TestPoint_Pad_1.0x1.0mm
- removed J7: Key 6, TestPoint:TestPoint_Pad_1.0x1.0mm
- removed J8: Key 7, TestPoint:TestPoint_Pad_1.0x1.0mm
- removed J9: Key 8, TestPoint:TestPoint_Pad_1.0x1.0mm
- moved RV1 43.2 mm to (135.0, 70.2), turned to 0 degrees
Routing:
- net (no net): track 121.4 -> 0.00 mm

Commit message: Updates to PCB
Parts:
- added G***: LOGO, LOGO, F.Cu at (113.0, 56.0)
- added J1: Conn_01x01_Male, Connector_Samtec_HPM_THT:Samtec_HPM-01-01-x-S_Straight_1x01_Pitch5.08mm, F.Cu at (109.0, 87.0)
- added R1: R, Resistor_SMD:R_1206_3216Metric, F.Cu at (125.4, 86.1)
- added R10: R, Resistor_SMD:R_1206_3216Metric, F.Cu at (150.8, 86.1)
- added R11: R, Resistor_SMD:R_1206_3216Metric, F.Cu at (153.9, 86.1)
- added R12: R, Resistor_SMD:R_1206_3216Metric, F.Cu at (157.1, 86.1)
- added R13: R, Resistor_SMD:R_1206_3216Metric, F.Cu at (160.3, 86.1)
- added R14: R, Resistor_SMD:R_1206_3216Metric, F.Cu at (163.4, 86.1)
- added R15: R, Resistor_SMD:R_1206_3216Metric, F.Cu at (166.6, 86.1)
- added R16: R, Resistor_SMD:R_1206_3216Metric, F.Cu at (169.8, 86.1)
- added R17: R, Resistor_SMD:R_1206_3216Metric, F.Cu at (172.9, 86.1)
- added R2: R, Resistor_SMD:R_1206_3216Metric, F.Cu at (128.6, 86.1)
- added R3: R, Resistor_SMD:R_1206_3216Metric, F.Cu at (131.7, 86.1)
- added R4: R, Resistor_SMD:R_1206_3216Metric, F.Cu at (134.9, 86.1)
- added R5: R, Resistor_SMD:R_1206_3216Metric, F.Cu at (138.1, 86.1)
- added R6: R, Resistor_SMD:R_1206_3216Metric, F.Cu at (141.2, 86.1)
- added R7: R, Resistor_SMD:R_1206_3216Metric, F.Cu at (122.2, 86.1)
- added R8: R, Resistor_SMD:R_1206_3216Metric, F.Cu at (144.4, 86.1)
- added R9: R, Resistor_SMD:R_1206_3216Metric, F.Cu at (147.6, 86.1)
- moved RV1 97.8 mm to (232.2, 80.0), turned to 90 degrees
Routing:
- net /AIN0: track 0.00 -> 49.1 mm
- net /Key2: track 0.00 -> 45.9 mm, vias 0 -> 2
- net /Key7: track 0.00 -> 44.6 mm, vias 0 -> 2
- net /Key14: track 0.00 -> 43.7 mm, vias 0 -> 2
- net /Key9: track 0.00 -> 43.0 mm, vias 0 -> 2
- net /Key1: track 0.00 -> 26.0 mm
- net /Key4: track 0.00 -> 25.8 mm
- net /Key0: track 0.00 -> 25.6 mm
- net /Key5: track 0.00 -> 25.4 mm
- net /Key13: track 0.00 -> 24.7 mm
- net /Key3: track 0.00 -> 24.4 mm
- net /Key12: track 0.00 -> 24.2 mm
- net /Key8: track 0.00 -> 24.1 mm
- net /Key11: track 0.00 -> 24.0 mm
- net /Key16: track 0.00 -> 23.6 mm
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- added copper zone on F.Cu, net /Key0
- added copper zone on F.Cu, net /Key1
- added copper zone on F.Cu, net /Key10
- added copper zone on F.Cu, net /Key11
- added copper zone on F.Cu, net /Key12
- added copper zone on F.Cu, net /Key13
- added copper zone on F.Cu, net /Key14
- added copper zone on F.Cu, net /Key15
- added copper zone on F.Cu, net /Key16
- added copper zone on F.Cu, net /Key2
- added copper zone on F.Cu, net /Key3
- added copper zone on F.Cu, net /Key4
- added copper zone on F.Cu, net /Key5
- added copper zone on F.Cu, net /Key6
- added copper zone on F.Cu, net /Key7
- added copper zone on F.Cu, net /Key8
- added copper zone on F.Cu, net /Key9
- removed copper zone on F.Cu, net (none)

Commit message: Updates
Parts:
- removed RV1: R_Potentiometer, Potentiometer_THT:Potentiometer_Bourns_PTA1543_Single_Slide
- added R18: COM-09806, Project:TRIM_COM-09806, F.Cu at (108.2, 86.8)
- J1: footprint Connector_Samtec_HPM_THT:Samtec_HPM-01-01-x-S_Straight_1x01_Pitch5.08mm -> Connector_Pin:Pin_D1.0mm_L10.0mm
- moved J1 44.6 mm to (153.5, 90.5)
- moved G*** 11.0 mm to (122.8, 51.0)
- moved R11 6.17 mm to (159.7, 84.0)
- moved R12 6.17 mm to (162.9, 84.0)
- moved R14 6.17 mm to (169.2, 84.0)
- moved R15 6.17 mm to (172.4, 84.0)
- moved R17 6.17 mm to (178.8, 84.0)
- moved R2 6.17 mm to (134.4, 84.0)
- moved R3 6.17 mm to (137.5, 84.0)
- moved R5 6.17 mm to (143.9, 84.0)
- moved R8 6.17 mm to (150.2, 84.0)
- moved R9 6.17 mm to (153.4, 84.0)
- moved R1 6.17 mm to (131.2, 84.0)
- moved R7 6.17 mm to (128.0, 84.0)
- moved R10 6.17 mm to (156.6, 84.0)
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Routing:
- net +1V8: track 0.00 -> 66.9 mm, vias 0 -> 1
- net /AIN1: track 0.00 -> 65.7 mm, vias 0 -> 1
- net GNDA: track 0.00 -> 59.8 mm, vias 0 -> 1
- net /AIN0: track 49.1 -> 69.0 mm
- net /Key4: track 25.8 -> 14.6 mm
- net /Key1: track 26.0 -> 14.8 mm
- net /Key2: track 45.9 -> 34.8 mm
- net /Key5: track 25.4 -> 14.3 mm
- net /Key8: track 24.1 -> 13.8 mm
- net /Key13: track 24.7 -> 14.9 mm
- net /Key10: track 23.5 -> 13.8 mm
- net /Key0: track 25.6 -> 16.0 mm
- net /Key12: track 24.2 -> 14.6 mm
- net /Key3: track 24.4 -> 15.1 mm
- net /Key7: track 44.6 -> 35.5 mm
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Other:
- board text added: "Logan Manthey 2024"
- board text added: "PCB3D_BR_test"
- board text added: "PCB3D_TL_test"

Commit message: Added Gerbers
Parts:
- removed J1: Conn_01x01_Male, Connector_Pin:Pin_D1.0mm_L10.0mm
- added ?: , , F.Cu at (153.5, 90.5)
Routing:
- net /Key9: track 35.1 -> 38.6 mm
- net /Key7: track 35.5 -> 39.0 mm
- net /Key2: track 34.8 -> 38.3 mm
- net /Key14: track 36.0 -> 39.5 mm
Other:
- board text added: "Keyboard Cape"
- board text removed: "Logan Manthey 2024"

Commit message: Updates to Readme
Other:
- board text removed: "Note: due to to way pin numbers work on the BBB, the connectors are actually 2.54mm pin headers with the 3D models overridden."
- board text removed: "PCB3D_BR_test"
- board text removed: "PCB3D_TL_test"
Changed lines of the file:
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@@
     (effects (font (size 3 3) (thickness 0.5) bold) (justify left bottom))
-  )
-  (gr_text "PCB3D_BR_test" (at 191 103) (layer "Dwgs.User")
-    (effects (font (size 1.5 1.5) (thickness 0.3) bold) (justify left bottom))
-  )
-  (gr_text "PCB3D_TL_test" (at 79 42) (layer "Dwgs.User")
-    (effects (font (size 1.5 1.5) (thickness 0.3) bold) (justify left bottom))
-  )
-  (gr_text "Note: due to to way pin numbers work on the BBB, the connectors\nare actually 2.54mm pin headers with the 3D models overridden." (at 101 103) (layer "Cmts.User")
-    (effects (font (size 1.5 1.5) (thickness 0.3)) (justify left))
   )
   (segment (start 119.5 87.75) (end 117.5 89.75) (width 1) (layer "F.Cu") (net 1))
